File: hw/usb2nrf.sch (KiCad schematic (older format))
At the start: 16 parts, among them IC1 ATMEGA8-AI, P1 CONN_01X03, P2 CONN_01X02, P3 CONN_01X06, P4 USBTTL, Y1 Crystal

Commit message: hw: update kicad version
Parts:
- removed D3: LED, LEDs:LED_0805_HandSoldering, symbol LED
- removed P3: CONN_01X06, Pin_Headers:Pin_Header_Straight_1x06_Pitch2.54mm, symbol CONN_01X06
- removed R3: R, Resistors_SMD:R_0805_HandSoldering, symbol R
- added C1, Cavr2, Clcd1, Cnrf1, Csrv3: 100n, Capacitors_SMD:C_0805, symbol Device:C
- added C4: 10u, Capacitors_ThroughHole:CP_Radial_D5.0mm_P2.00mm, symbol Device:CP
- added C5, Cavr3, Clcd2, Cnrf2, Csrv1: 10u, Capacitors_SMD:C_1210, symbol Device:CP
- added CON1: AVR-JTAG-10, Pin_Headers:Pin_Header_Straight_2x05_Pitch2.54mm, symbol atmel:AVR-JTAG-10
- added D5, D6, D7: LED, LEDs:LED_0805, symbol Device:LED
- added P3, P6: CONN_01X01, Pin_Headers:Pin_Header_Straight_1x01_Pitch2.54mm, symbol conn:CONN_01X01
- added P5: LCD_CONN, lcd_n1202:SIL-12, symbol conn:CONN_01X12
- added Pnrf1: nrf_test, Pin_Headers:Pin_Header_Straight_1x07_Pitch2.54mm, symbol conn:CONN_01X07
- added Psrv1: CONN_srv, Pin_Headers:Pin_Header_Straight_1x03_Pitch2.54mm, symbol conn:CONN_01X03
- added Puart1: uart_test, Pin_Headers:Pin_Header_Straight_1x03_Pitch2.54mm, symbol conn:CONN_01X03
- added R10, R14, R15, R3, R9: 10k, Resistors_SMD:R_0805, symbol Device:R
- added R11, R4, R5, R6: R, Resistors_SMD:R_0805, symbol Device:R
- added R12: 47k, Resistors_SMD:R_0805, symbol Device:R
- added R13, R16: 511, Resistors_SMD:R_0805, symbol Device:R
- added R7, R8: 150, Resistors_SMD:R_0805, symbol Device:R
- added SW1, SW2, SWrst1: SW_Push, Buttons_Switches_ThroughHole:SW_PUSH_6mm_h4.3mm, symbol Switch:SW_Push
- added SW3: Rotary_Encoder_Switch, misc:encoder, symbol Device:Rotary_Encoder_Switch
- added U1: AMS1117-3.3, TO_SOT_Packages_SMD:SOT-223-3_TabPin2, symbol Regulator_Linear:AMS1117-3.3
- C2, C3: value C -> 22p; footprint Capacitors_SMD:C_0805_HandSoldering -> Capacitors_SMD:C_0805; symbol C -> Device:C
- Cavr1: renamed from C1; footprint Capacitors_SMD:C_0805_HandSoldering -> Capacitors_SMD:C_0805; symbol C -> Device:C
- D1, D2: footprint LEDs:LED_0805_HandSoldering -> LEDs:LED_0805; symbol LED -> usb2nrf-rescue:LED
- IC1: symbol ATMEGA8-AI -> atmel:ATMEGA8-AI
- NRF24L1: renamed from D4; symbol NRF24L01 -> modules:NRF24L01
- P1: symbol CONN_01X03 -> conn:CONN_01X03
- P2: symbol CONN_01X02 -> conn:CONN_01X02
- P4: symbol CONN_01X05 -> conn:CONN_01X05
- R1, R2: footprint Resistors_SMD:R_0805_HandSoldering -> Resistors_SMD:R_0805; symbol R -> Device:R
- Y1: value Crystal -> 16M; symbol Crystal -> Device:Crystal
Connections:
- net 3v3: now also C5.1, Cavr2.1, Cavr3.1, Clcd1.2, Clcd2.1, Cnrf1.2, Cnrf2.1, D5.2 (A), D6.2 (A), D7.2 (A), P5.7 (P7), P5.8 (P8), R11.2, R12.1, R13.1, R16.1, SW1.2, SW2.2, U1.2 (VO); no longer P4.1 (P1)
- net 5v: now also C4.1, CON1.2, Csrv1.1, Csrv3.1, Psrv1.2 (P2), U1.3 (VI)
- net ce: now also Pnrf1.2 (P2)
- net csn: now also Pnrf1.3 (P3)
- net irq: now also Pnrf1.7 (P7)
- net lcd_clk: now also P5.6 (P6)
- net lcd_cs: now also P5.3 (P3)
- net lcd_rst: now also P5.2 (P2)
- net lcd_sda: now also P5.5 (P5)
- net miso: now also CON1.9, Pnrf1.6 (P6)
- net mosi: now also CON1.1, Pnrf1.5 (P5)
- net reset: now also P2.2 (P2), C1.1, CON1.5, R12.2, SWrst1.1; no longer P2.1 (P1)
- net rx_usb: now also Puart1.3 (P3), R6.1
- net sck: now also CON1.7, Pnrf1.4 (P4)
- net tx_usb: now also Puart1.2 (P2), R5.1
- net at IC1.1 ((INT1)PD3): now also R8.2
- net at IC1.2 ((XCK/T0)PD4): now also Psrv1.3 (P3)
- net at IC1.23 ((ADC0)PC0): now also R3.1, SW3.A
- net at IC1.24 ((ADC1)PC1): now also R14.1, SW3.B
- net at IC1.32 ((INT0)PD2): now also R7.2
- net enc_btn: now reaches IC1.9 ((T1)PD5)
- net enc_btn: now also R15.1, SW3.S2
- net gnd renamed GNDPWR
- net GNDPWR: now also P2.1 (P1), C1.2, C4.2, C5.2, CON1.10, CON1.4, CON1.6, CON1.8, Cavr2.2, Cavr3.2, Clcd1.1, Clcd2.2, Cnrf1.1, Cnrf2.2, Csrv1.2, Csrv3.2, P5.10 (P10), P5.4 (P4), P5.9 (P9), Pnrf1.1 (P1), Psrv1.1 (P1), Puart1.1 (P1), R10.1, R14.2, R15.2, R3.2, R4.2, R9.2, SWrst1.2, U1.1 (GND); no longer P2.2 (P2)
- new net: R7.1, R9.1, SW1.1
- new net: R10.2, R8.1, SW2.1
- new net: D5.1 (K), R4.1
- new net: D6.1 (K), R5.2
- new net: D7.1 (K), R6.2
- new net: R13.2, SW3.C
- new net: R16.2, SW3.S1
- new net lcd_backlight: P5.11 (P11), R11.1
- no-connect marks 8 -> 9
Other:
- moved on the sheet: C2, C3, Cavr1, NRF24L1, P1, P2, P4
